Commit message: Added Gazebo elements

File: description/robot_core.xacro (robot description, xacro)
@@ -44,4 +44,7 @@
         </xacro:inertial_box>
     </link>
+    <gazebo reference="chassis">
+        <material>Gazebo/White</material>
+    </gazebo>
     <!-- Left Wheel link-->
     <joint name="left_wheel_joint" type="continuous">
@@ -67,4 +70,7 @@
         </xacro:inertial_cylinder>
     </link>
+    <gazebo reference="left_wheel">
+        <material>Gazebo/Blue</material>
+    </gazebo>
     <!-- Right Wheel Link-->
     <joint name="right_wheel_joint" type="continuous">
@@ -90,4 +96,7 @@
         </xacro:inertial_cylinder>
     </link>
+    <gazebo reference="right_wheel">
+        <material>Gazebo/Blue</material>
+    </gazebo>
     <!-- Caster Wheel link-->
     <joint name="caster_wheel_joint" type="fixed">
@@ -113,3 +122,8 @@
         </xacro:inertial_sphere>
     </link>
+    <gazebo reference="caster_wheel">
+        <material>Gazebo/Black</material>
+        <mu1 value="0.001"/>
+        <mu2 value="0.001"/>
+    </gazebo>
 </robot>
